Commit message: robot_done

File: src/ur_description/urdf/common.gazebo.xacro (robot description, xacro)
@@ -6,5 +6,4 @@
       <!--robotSimType>gazebo_ros_control/DefaultRobotHWSim</robotSimType-->
     </plugin>
-<!--
     <plugin name="gazebo_ros_power_monitor_controller" filename="libgazebo_ros_power_monitor.so">
       <alwaysOn>true</alwaysOn>
@@ -19,5 +18,4 @@
       <chargeVoltage>16.41</chargeVoltage>
     </plugin>
--->
   </gazebo>
 </robot>

File: src/ur_description/urdf/kinect_sensor.urdf.xacro (robot description, xacro)
@@ -2,9 +2,9 @@
 <robot xmlns:xacro="http://wiki.ros.org/xacro"  name="kinect_camera" >
     <link name="camera_support">
-    <inertial>
-      <origin xyz="0 0 0.5" rpy="0 0 0"/>
-      <mass value="20"/>
-      <inertia ixx="200" ixy="200" ixz="200" iyy="200" iyz="200" izz="200"/>
-     </inertial>
+      <inertial>
+        <origin xyz="0 0 0.5" rpy="0 0 0"/>
+       <mass value="20"/>
+       <inertia ixx="200" ixy="200" ixz="200" iyy="200" iyz="200" izz="200"/>
+      </inertial>
      <visual>
        <origin xyz="0 0 0.5" rpy="0 0 0"/>
@@ -45,5 +45,5 @@
     </inertial>
   </link>
- <joint name="camera_support" type="fixed">
+<joint name="camera_support" type="fixed">
     <axis xyz="0 1 0" />
     <origin xyz="0 2.5 -0.2" rpy="0 0 -3.14"/>
@@ -73,5 +73,5 @@
       <material>Gazebo/Orange</material>
      </gazebo>
-   <xacro:property name="link_name" value="camera_link" />
+<xacro:property name="link_name" value="camera_link" />
  <xacro:property name="camera_name" value="3Dcamera" />
  <xacro:property name="frame_name" value="camera_optical_link" />

File: src/ur_description/urdf/test_jean.urdf (robot description, URDF)
Before this commit: robot test_jean, 3 links, 2 joints
Links:
- removed link base0_link
- removed link jean
- added link cabin, mass 35.9737389131107; collision mesh filename=package://ur_description/meshes/cabin.stl; visual mesh filename=package://ur_description/meshes/cabin.dae scale=15 30 20
Joints:
- removed joint pant_link
- joint world_link: axis 0 0 1 -> (none); child base0_link -> cabin; origin xyz=-0.498714986842488 -0.0904135841410607 0 rpy=-1.5707963267949 0.00437080591465176 0 -> xyz=0.5 0.5 0 rpy=-1.570796327 3.141592654 -4.71238898

File: src/ur_description/urdf/ur5_joint_limited_robot.urdf.xacro (robot description, xacro)
@@ -3,5 +3,5 @@
        name="ur5" >
   <xacro:arg name="transmission_hw_interface" default="hardware_interface/PositionJointInterface"/>
-  <xacro:property name="camera_link" value="0.05" />
+  <!--<xacro:property name="camera_link" value="0.05" />-->
   <!-- common stuff -->
   <xacro:include filename="$(find ur_description)/urdf/common.gazebo.xacro" />
@@ -19,5 +19,5 @@
   />
   <link name="world" />
-    <link name="pedestal">
+    <link name="support">
     <inertial>
       <origin xyz="0 0 0.5" rpy="0 0 0"/>
@@ -28,5 +28,6 @@
        <origin xyz="0 0 0.5" rpy="0 0 0"/>
        <geometry>
-         <cylinder radius="0.1" length="1.0" />
+        <box size='0.5 0.5 1'/>
+         <!--<cylinder radius="0.1" length="1.0" />-->
        </geometry>
        <material name="Gray">
@@ -41,19 +42,17 @@
       </collision>
     </link>
-    <gazebo reference="pedestal">
-      <mu1>0.2</mu1>
-      <mu2>0.2</mu2>
-      <material>Gazebo/Orange</material>
+    <gazebo reference="support">
+      <material>Gazebo/Grey</material>
      </gazebo>
    <joint name="world_joint" type="fixed">
     <parent link="world" />
-    <child link = "pedestal" />
+    <child link = "support" />
     <origin xyz="0.0 0.0 -0.1" rpy="0.0 0.0 0.0" />
     </joint>
  <joint name="base_joint" type="fixed">
-    <parent link="pedestal" />
+    <parent link="support" />
     <child link = "base_link" />
     <origin xyz="0.0 0.0 1.0" rpy="0.0 0.0 0.0" />
-    </joint>
-<xacro:include filename="$(find ur_description)/urdf/kinect_sensor.urdf.xacro" />
+  </joint>
+<!--xacro:include filename="$(find ur_description)/urdf/kinect_sensor.urdf.xacro" /> -->
 </robot>
